File: EDA/berlin.kicad_pcb (KiCad board)
At the start: 0 parts

Commit message: initial pcb layouting
Parts:
- added ?: , , F.Cu at (350.8, 69.8)
- added REF**: Potentiometer_Bourns_PTA6043_Single_Slide, Potentiometer_THT:Potentiometer_Bourns_PTA6043_Single_Slide, F.Cu at (61.7, 68.1)
- added REF**: EA_DOGXL160-7_Backlight, Display:EA_DOGXL160-7_Backlight, F.Cu at (441.3, 60.5)
- added REF**: Potentiometer_Bourns_PTA6043_Single_Slide, Potentiometer_THT:Potentiometer_Bourns_PTA6043_Single_Slide, F.Cu at (242.8, 68.1)
- added REF**: Potentiometer_Bourns_PTA6043_Single_Slide, Potentiometer_THT:Potentiometer_Bourns_PTA6043_Single_Slide, F.Cu at (152.3, 68.1)
- added SW1: MXSwitch, acheron_MX:MX100, B.Cu at (41.2, 108.0)
- added SW10: MXSwitch, acheron_MX:MX100, B.Cu at (69.8, 155.6)
- added SW100: MXSwitch, acheron_MX:MX100, B.Cu at (369.9, 108.0)
- added SW101: MXSwitch, acheron_MX:MX100, B.Cu at (393.7, 136.6)
- added SW102: MXSwitch, acheron_MX:MX100, B.Cu at (393.7, 155.6)
- added SW103: MXSwitch, acheron_MX:MX100, B.Cu at (393.7, 174.7)
- added SW104: MXSwitch, acheron_MX:MX100, B.Cu at (393.7, 193.7)
- added SW105-1: MXSwitch, acheron_MX:MX200, B.Cu at (403.2, 212.8)
- added SW105-2: MXSwitch, acheron_MX:MX100, B.Cu at (393.7, 212.8)
- added SW106: MXSwitch, acheron_MX:MX100, B.Cu at (331.8, 136.5)
- added SW107: MXSwitch, acheron_MX:MX100, B.Cu at (331.8, 155.6)
- added SW108: MXSwitch, acheron_MX:MX100, B.Cu at (412.7, 136.6)
- added SW109: MXSwitch, acheron_MX:MX100, B.Cu at (412.7, 155.6)
- added SW11: MXSwitch, acheron_MX:MX100, B.Cu at (74.6, 174.7)
- added SW110: MXSwitch, acheron_MX:MX100, B.Cu at (412.7, 174.7)
- added SW111: MXSwitch, acheron_MX:MX100, B.Cu at (412.7, 193.7)
- added SW112: MXSwitch, acheron_MX:MX100, B.Cu at (412.7, 212.8)
- added SW113: MXSwitch, acheron_MX:MX100, B.Cu at (350.8, 136.5)
- added SW114: MXSwitch, acheron_MX:MX100, B.Cu at (350.8, 155.6)
- added SW115: MXSwitch, acheron_MX:MX100, B.Cu at (431.8, 136.6)
- added SW116: MXSwitch, acheron_MX:MX100, B.Cu at (431.8, 155.6)
- added SW117: MXSwitch, acheron_MX:MX100, B.Cu at (431.8, 174.7)
- added SW118: MXSwitch, acheron_MX:MX100, B.Cu at (431.8, 193.7)
- added SW119: MXSwitch, acheron_MX:MX100, B.Cu at (431.8, 212.8)
- added SW12: MXSwitch, acheron_MX:MX100, B.Cu at (65.1, 193.7)
- added SW120: MXSwitch, acheron_MX:MX100, B.Cu at (369.9, 136.5)
- added SW121: MXSwitch, acheron_MX:MX100, B.Cu at (369.9, 155.6)
- added SW122: MXSwitch, acheron_MX:MX100, B.Cu at (450.8, 136.6)
- added SW123: MXSwitch, Acheron_MX:MX100, B.Cu at (450.8, 174.7)
- added SW124-1: MXSwitch, acheron_MX:MX200, B.Cu at (450.8, 165.2)
- added SW124-2: MXSwitch, Acheron_MX:MX100, B.Cu at (450.8, 155.6)
- added SW125: MXSwitch, acheron_MX:MX200R, B.Cu at (450.8, 203.3)
- added SW126: Rotary_Encoder_Switch_Chassis, acheronHardware:ALPS_EC11E, F.Cu at (41.3, 76.2)
- added SW126: Rotary_Encoder_Switch_Chassis, acheronHardware:ALPS_EC11E, F.Cu at (369.9, 69.8)
- added SW129: MXSwitch, acheron_MX:MX275, B.Cu at (291.3, 193.7)
- added SW13: MXSwitch, acheron_MX:MX125, B.Cu at (67.4, 212.8)
- added SW14: MXSwitch, acheron_MX:MX100, B.Cu at (88.9, 88.9)
- added SW15: MXSwitch, acheron_MX:MX100, B.Cu at (88.9, 108.0)
- added SW16: MXSwitch, acheron_MX:MX100, B.Cu at (79.3, 136.6)
- added SW17: MXSwitch, acheron_MX:MX100, B.Cu at (88.9, 155.6)
- added SW18: MXSwitch, acheron_MX:MX100, B.Cu at (93.6, 174.7)
- added SW19: MXSwitch, acheron_MX:MX100, B.Cu at (84.1, 193.7)
- added SW2: MXSwitch, acheron_MX:MX100, B.Cu at (41.2, 136.6)
- added SW20-1: MXSwitch, acheron_MX:MX125, B.Cu at (257.9, 212.8)
- added SW20-1: MXSwitch, acheron_MX:MX125, B.Cu at (281.7, 212.8)
- added SW20-1: MXSwitch, acheron_MX:MX125, B.Cu at (305.6, 212.8)
- added SW20-1: MXSwitch, acheron_MX:MX125, B.Cu at (234.1, 212.8)
- added SW21: MXSwitch, acheron_MX:MX100, B.Cu at (107.9, 88.9)
- added SW22: MXSwitch, acheron_MX:MX100, B.Cu at (107.9, 108.0)
- added SW23: MXSwitch, acheron_MX:MX100, B.Cu at (98.4, 136.6)
- added SW24: MXSwitch, acheron_MX:MX100, B.Cu at (107.9, 155.6)
- added SW25: MXSwitch, acheron_MX:MX100, B.Cu at (112.7, 174.7)
- added SW26: MXSwitch, acheron_MX:MX100, B.Cu at (103.2, 193.7)
- added SW27: MXSwitch, acheron_MX:MX100, B.Cu at (127.0, 88.9)
- added SW28: MXSwitch, acheron_MX:MX100, B.Cu at (127.0, 108.0)
- added SW29: MXSwitch, acheron_MX:MX100, B.Cu at (117.4, 136.6)
- added SW3: MXSwitch, acheron_MX:MX150, B.Cu at (46.0, 155.6)
- added SW30: MXSwitch, acheron_MX:MX100, B.Cu at (127.0, 155.6)
- added SW31: MXSwitch, acheron_MX:MX100, B.Cu at (131.7, 174.7)
- added SW32: MXSwitch, acheron_MX:MX100, B.Cu at (122.2, 193.7)
- added SW33: MXSwitch, acheron_MX:MX100, B.Cu at (160.4, 88.9)
- added SW34: MXSwitch, acheron_MX:MX100, B.Cu at (160.4, 108.0)
- added SW35: MXSwitch, acheron_MX:MX100, B.Cu at (136.5, 136.6)
- added SW36: MXSwitch, acheron_MX:MX100, B.Cu at (146.0, 155.6)
- added SW37: MXSwitch, acheron_MX:MX100, B.Cu at (150.8, 174.7)
- added SW38: MXSwitch, acheron_MX:MX100, B.Cu at (141.3, 193.7)
- added SW39-1: MXSwitch, acheron_MX:MX625, B.Cu at (162.7, 212.8)
- added SW39-3: MXSwitch, acheron_MX:MX125, B.Cu at (91.2, 212.8)
- added SW4-2: MXSwitch, Acheron_MX:MX175, B.Cu at (48.4, 174.7)
- added SW40: MXSwitch, acheron_MX:MX100, B.Cu at (179.5, 88.9)
- added SW41: MXSwitch, acheron_MX:MX100, B.Cu at (179.5, 108.0)
- added SW42: MXSwitch, acheron_MX:MX100, B.Cu at (155.5, 136.6)
- added SW43: MXSwitch, acheron_MX:MX100, B.Cu at (165.1, 155.6)
- added SW44: MXSwitch, acheron_MX:MX100, B.Cu at (169.8, 174.7)
- added SW45: MXSwitch, acheron_MX:MX100, B.Cu at (160.3, 193.7)
- added SW46: MXSwitch, acheron_MX:MX100, B.Cu at (198.5, 88.9)
- added SW47: MXSwitch, acheron_MX:MX100, B.Cu at (198.5, 108.0)
- added SW48: MXSwitch, acheron_MX:MX100, B.Cu at (174.6, 136.6)
- added SW49: MXSwitch, acheron_MX:MX100, B.Cu at (184.1, 155.6)
- added SW5-1: MXSwitch, acheron_MX:MX125, B.Cu at (43.6, 193.7)
- added SW50: MXSwitch, acheron_MX:MX100, B.Cu at (188.9, 174.7)
- added SW51: MXSwitch, acheron_MX:MX100, B.Cu at (179.4, 193.7)
- added SW52: MXSwitch, acheron_MX:MX100, B.Cu at (217.6, 88.9)
- added SW53: MXSwitch, acheron_MX:MX100, B.Cu at (217.6, 108.0)
- added SW54: MXSwitch, acheron_MX:MX100, B.Cu at (193.6, 136.6)
- added SW55: MXSwitch, acheron_MX:MX100, B.Cu at (203.2, 155.6)
- added SW56: MXSwitch, acheron_MX:MX100, B.Cu at (207.9, 174.7)
- added SW57: MXSwitch, acheron_MX:MX100, B.Cu at (198.4, 193.7)
- added SW58: MXSwitch, acheron_MX:MX100, B.Cu at (250.8, 88.9)
- added SW59: MXSwitch, acheron_MX:MX100, B.Cu at (250.8, 108.0)
- added SW6-1: MXSwitch, acheron_MX:MX125, B.Cu at (43.6, 212.8)
- added SW60: MXSwitch, acheron_MX:MX100, B.Cu at (212.7, 136.6)
- added SW61: MXSwitch, acheron_MX:MX100, B.Cu at (222.2, 155.6)
- added SW62: MXSwitch, acheron_MX:MX100, B.Cu at (227.0, 174.7)
- added SW63: MXSwitch, acheron_MX:MX100, B.Cu at (217.5, 193.7)
- added SW65: MXSwitch, acheron_MX:MX100, B.Cu at (269.8, 88.9)
- added SW66: MXSwitch, acheron_MX:MX100, B.Cu at (269.8, 108.0)
- added SW67: MXSwitch, acheron_MX:MX100, B.Cu at (231.7, 136.6)
- added SW68: MXSwitch, acheron_MX:MX100, B.Cu at (241.3, 155.6)
- added SW69: MXSwitch, acheron_MX:MX100, B.Cu at (246.0, 174.7)
- added SW7: MXSwitch, acheron_MX:MX100, B.Cu at (69.8, 88.9)
- added SW70: MXSwitch, acheron_MX:MX100, B.Cu at (236.5, 193.7)
- added SW72: MXSwitch, acheron_MX:MX100, B.Cu at (288.9, 88.9)
- added SW73: MXSwitch, acheron_MX:MX100, B.Cu at (288.9, 108.0)
- added SW74: MXSwitch, acheron_MX:MX100, B.Cu at (250.8, 136.6)
- added SW75: MXSwitch, acheron_MX:MX100, B.Cu at (260.3, 155.6)
- added SW76: MXSwitch, acheron_MX:MX100, B.Cu at (265.1, 174.7)
- added SW77: MXSwitch, acheron_MX:MX100, B.Cu at (255.6, 193.7)
- added SW79: MXSwitch, acheron_MX:MX100, B.Cu at (307.9, 88.9)
- added SW8: MXSwitch, acheron_MX:MX100, B.Cu at (69.8, 108.0)
- added SW80: MXSwitch, acheron_MX:MX100, B.Cu at (307.9, 108.0)
- added SW81: MXSwitch, acheron_MX:MX100, B.Cu at (269.8, 136.6)
- added SW82: MXSwitch, acheron_MX:MX100, B.Cu at (279.4, 155.6)
- added SW83: MXSwitch, acheron_MX:MX100, B.Cu at (284.1, 174.7)
- added SW85: MXSwitch, acheron_MX:MX100, B.Cu at (331.8, 212.8)
- added SW86: MXSwitch, acheron_MX:MX100, B.Cu at (331.8, 69.8)
- added SW86: MXSwitch, acheron_MX:MX100, B.Cu at (331.8, 88.9)
- added SW87: MXSwitch, acheron_MX:MX100, B.Cu at (331.8, 108.0)
- added SW88-2: MXSwitch, acheron_MX:MX200, B.Cu at (298.4, 136.6)
- added SW9: MXSwitch, acheron_MX:MX100, B.Cu at (60.3, 136.6)
- added SW90-2: MXSwitch, acheron_MX:MX_ISOEnter, B.Cu at (305.6, 165.1)
- added SW91: MXSwitch, acheron_MX:MX100, B.Cu at (350.8, 193.7)
- added SW92: MXSwitch, acheron_MX:MX100, B.Cu at (350.8, 212.8)
- added SW93: MXSwitch, acheron_MX:MX100, B.Cu at (350.8, 88.9)
- added SW93: MXSwitch, acheron_MX:MX100, B.Cu at (350.8, 69.8)
- added SW94: MXSwitch, acheron_MX:MX100, B.Cu at (350.8, 108.0)
- added SW98: MXSwitch, acheron_MX:MX100, B.Cu at (369.9, 212.8)
- added SW99: MXSwitch, acheron_MX:MX100, B.Cu at (369.9, 88.9)
Other:
- copper layers 0 -> 2
