File: EDA/berlin.kicad_pcb (KiCad board)
At the start: 2 copper layers, 129 parts, among them SW1,1 Rotary_Encoder_Switch_Chassis, SW1,10 MXSwitch, SW1,11 MXSwitch, SW1,12 MXSwitch, SW1,13 MXSwitch, SW1,14 MXSwitch, SW1,15 MXSwitch, SW1,16 Rotary_Encoder_Switch_Chassis, SW1,2 MXSwitch, SW1,3 MXSwitch, SW1,4 MXSwitch, SW1,5 MXSwitch, SW1,6 MXSwitch, SW1,7 MXSwitch, SW1,8 MXSwitch, SW1,9 MXSwitch, SW125 2,19, SW2,1 MXSwitch, SW2,10 MXSwitch, SW2,11 MXSwitch, SW2,12 MXSwitch, SW2,13 MXSwitch, SW2,14 MXSwitch, SW2,15 MXSwitch, SW2,16 MXSwitch, SW2,17 MXSwitch, SW2,18 MXSwitch, SW2,2 MXSwitch, SW2,3 MXSwitch, SW2,4 MXSwitch, SW2,5 MXSwitch, SW2,6 MXSwitch, SW2,7 MXSwitch, SW2,8 MXSwitch, SW2,9 MXSwitch, SW3,1 MXSwitch, SW3,10 MXSwitch, SW3,11 MXSwitch, SW3,12 MXSwitch, SW3,13 MXSwitch, SW3,14 MXSwitch, SW3,15 MXSwitch, SW3,16 MXSwitch, SW3,17 MXSwitch, SW3,18 MXSwitch, SW3,19 MXSwitch, SW3,2 MXSwitch, SW3,3 MXSwitch, SW3,4 MXSwitch, SW3,5 MXSwitch, SW3,6 MXSwitch, SW3,7 MXSwitch, SW3,8 MXSwitch, SW3,9 MXSwitch, SW4,1 MXSwitch, SW4,10 MXSwitch, SW4,11 MXSwitch, SW4,12 MXSwitch, SW4,13 MXSwitch, SW4,14 MXSwitch, SW4,15 MXSwitch, SW4,16 MXSwitch, SW4,17 MXSwitch, SW4,18 MXSwitch, SW4,19 MXSwitch, SW4,2 MXSwitch, SW4,3 MXSwitch, SW4,4 MXSwitch, SW4,5 MXSwitch, SW4,6 MXSwitch, SW4,7 MXSwitch, SW4,8 MXSwitch, SW4,9 MXSwitch, SW5,1 MXSwitch, SW5,10 MXSwitch, SW5,11 MXSwitch, SW5,12 MXSwitch, SW5,13 MXSwitch, SW5,14 MXSwitch, SW5,15 MXSwitch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

Commit message: add hotswap switches
Parts:
- added D94: 1N4148, acheronComponents:D_SOD-123, B.Cu at (52.7, 108.0)
- added J705: TYPE-C-31-M12_13, acheronConnectors:TYPE-C-31-M-12, B.Cu at (143.5, 58.1)
- added REF**: LQFP100-14X14mm, 2021-09-09_19-40-16:STM32F072VBT6, B.Cu at (234.3, 117.5)
- SW1,10, SW1,11, SW1,12, SW1,13, SW1,14, SW1,15, SW1,2, SW1,3, SW1,4, SW1,5, SW1,6, SW1,7, SW1,8, SW1,9, SW2,1, SW2,10, SW2,11, SW2,12, SW2,13, SW2,14, SW2,15, SW2,16, SW2,17, SW2,2, SW2,3, SW2,4, SW2,5, SW2,6, SW2,7, SW2,8, SW2,9, SW3,1, SW3,10, SW3,11, SW3,12, SW3,13, SW3,14, SW3,15, SW3,16, SW3,17, SW3,18, SW3,19, SW3,2, SW3,3, SW3,4, SW3,5, SW3,6, SW3,7, SW3,8, SW3,9, SW4,10, SW4,11, SW4,12, SW4,14, SW4,15, SW4,16, SW4,17, SW4,18, SW4,19, SW4,2, SW4,3, SW4,4, SW4,5, SW4,6, SW4,7, SW4,8, SW4,9, SW5,10, SW5,11, SW5,12, SW5,13, SW5,14, SW5,15, SW5,16, SW5,17, SW5,18, SW5,19, SW5,2, SW5,3, SW5,4, SW5,5, SW5,6, SW5,7, SW5,8, SW5,9, SW6,10, SW6,11, SW6,12, SW6,15, SW6,17, SW6,18, SW6,19, SW6,2, SW6,3, SW6,4, SW6,5, SW6,6, SW6,7, SW6,8, SW6,9, SW7,12, SW7,14, SW7,15, SW7,16, SW7,19: footprint acheron_MX:MX100 -> acheron_MXH:MX100H
- SW125: footprint acheron_MX:MX200R -> acheron_MXH:MX200HR
- SW2,18, SW4,13, SW7,17: footprint acheron_MX:MX200 -> acheron_MXH:MX200H
- SW4,1: footprint acheron_MX:MX150 -> acheron_MXH:MX150H
- SW5,1: footprint Acheron_MX:MX175 -> acheron_MXH:MX175H
- SW6,1, SW7,1, SW7,10, SW7,11, SW7,2, SW7,3, SW7,8, SW7,9: footprint acheron_MX:MX125 -> acheron_MXH:MX125H
- SW6,13: footprint acheron_MX:MX_ISOEnter -> acheron_MXH:MX_ISOEnterH
- SW7,13: footprint acheron_MX:MX275 -> acheron_MXH:MX275H
- SW7,6: footprint acheron_MX:MX625 -> acheron_MXH:MX625H
- moved REF** 69.4 mm to (441.3, 59.8), turned to -90 degrees
Routing:
- net (no net): track 0.00 -> 7.11 mm
- added copper zone on F.Cu, net (none)
