File: EDA/berlin.kicad_pcb (KiCad board)
At the start: 2 copper layers, 381 parts, among them J1 TYPE-C-31-M12_13, SW1,1 Rotary_Encoder_Switch_Chassis, SW1,10 MXSwitch, SW1,11 MXSwitch, SW1,12 MXSwitch, SW1,13 MXSwitch, SW1,14 MXSwitch, SW1,15 MXSwitch, SW1,16 Rotary_Encoder_Switch_Chassis, SW1,2 MXSwitch, SW1,3 MXSwitch, SW1,4 MXSwitch, SW1,5 MXSwitch, SW1,6 MXSwitch, SW1,7 MXSwitch, SW1,8 MXSwitch, SW1,9 MXSwitch, SW2,1 MXSwitch, SW2,10 MXSwitch, SW2,11 MXSwitch, SW2,12 MXSwitch, SW2,13 MXSwitch, SW2,14 MXSwitch, SW2,15 MXSwitch, SW2,16 MXSwitch, SW2,17 MXSwitch, SW2,18 MXSwitch, SW2,19 2,19, SW2,2 MXSwitch, SW2,3 MXSwitch, SW2,4 MXSwitch, SW2,5 MXSwitch, SW2,6 MXSwitch, SW2,7 MXSwitch, SW2,8 MXSwitch, SW2,9 MXSwitch, SW3,1 MXSwitch, SW3,10 MXSwitch, SW3,11 MXSwitch, SW3,12 MXSwitch, SW3,13 MXSwitch, SW3,14 MXSwitch, SW3,15 MXSwitch, SW3,16 MXSwitch, SW3,17 MXSwitch, SW3,18 MXSwitch, SW3,19 MXSwitch, SW3,2 MXSwitch, SW3,3 MXSwitch, SW3,4 MXSwitch, SW3,5 MXSwitch, SW3,6 MXSwitch, SW3,7 MXSwitch, SW3,8 MXSwitch, SW3,9 MXSwitch, SW4,1 MXSwitch, SW4,10 MXSwitch, SW4,11 MXSwitch, SW4,12 MXSwitch, SW4,13 MXSwitch, SW4,14 MXSwitch, SW4,15 MXSwitch, SW4,16 MXSwitch, SW4,17 MXSwitch, SW4,18 MXSwitch, SW4,19 MXSwitch, SW4,2 MXSwitch, SW4,3 MXSwitch, SW4,4 MXSwitch, SW4,5 MXSwitch, SW4,6 MXSwitch, SW4,7 MXSwitch, SW4,8 MXSwitch, SW4,9 MXSwitch, SW5,1 MXSwitch, SW5,10 MXSwitch, SW5,11 MXSwitch, SW5,12 MXSwitch, SW5,13 MXSwitch, SW5,14 MXSwitch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

Commit message: morte routing than the telekom will ever do
Connections:
- SW6,7 pad 1: (no net) -> Col7
Routing:
- net Col4: track 198.0 -> 265.5 mm
- net Col6: track 194.2 -> 181.9 mm
- net Col7: track 205.9 -> 201.3 mm
- net Col9: track 249.6 -> 251.6 mm
- net Col8: track 261.5 -> 260.9 mm

Commit message: still a better lovestory than twilight
Other:
- board outline added: 431.8 x 173.4 mm
Changed lines of the file:
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@@
   )
   (gr_line (start 462.28 57.785) (end 462.915 58.42) (layer "F.Cu") (width 0.2))
+  (gr_poly
+    (pts
+      (xy 149.225 57.785)
+      (xy 462.915 57.785)
+      (xy 462.915 224.79)
+      (xy 31.115 224.79)
+      (xy 31.115 57.785)
+      (xy 137.795 57.785)
+      (xy 137.795 51.435)
+      (xy 149.225 51.435)
+    ) (layer "B.Cu") (width 0.2) (fill none))
   (gr_rect (start 462.915 224.79) (end 30.734 57.785) (layer "Dwgs.User") (width 0.15) (fill none))
   (gr_rect (start 149.225 48.895) (end 137.795 57.785) (layer "Dwgs.User") (width 0.15) (fill none))
+  (gr_poly
+    (pts
+      (xy 149.225 57.785)
+      (xy 462.915 57.785)
+      (xy 462.915 224.79)
+      (xy 31.115 224.79)
+      (xy 31.115 57.785)
+      (xy 137.795 57.785)
+      (xy 137.795 51.435)
+      (xy 149.225 51.435)
+    ) (layer "Edge.Cuts") (width 0.1) (fill none))
   (segment (start 33.02 131.698) (end 33.02 133.1595) (width 0.25) (layer "B.Cu") (net 0))
   (segment (start 142.20825 153.06675) (end 138.65225 153.06675) (width 0.2) (layer "B.Cu") (net 0))

Commit message: update col traces
Parts:
- moved D36 8.34 mm to (305.6, 170.7)
Routing:
- net Col13: track 220.1 -> 211.1 mm
- net Col11: track 254.5 -> 245.7 mm
- net Col12: track 186.7 -> 178.7 mm
- net Col14: track 160.7 -> 167.3 mm
- net Col15: track 167.8 -> 173.5 mm
- net Col16: track 158.0 -> 161.3 mm
- net Col18: track 153.2 -> 155.5 mm
- net Col19: track 106.9 -> 109.3 mm
- net Col17: track 172.9 -> 175.2 mm

Commit message: update neopixels to reverse mount
Parts:
- D36 (x122): footprint acheron_Components:LED_WS2812B_5.0x5.0mm_P3.2mm -> acheron_Components:SK6812MINI_3535_6028_3.2x2.8mm_Round

Commit message: resolve drc conflicts
Parts:
- moved D36 3.51 mm to (446.3, 161.8)
- moved D36 0.61 mm to (445.1, 203.5)
- moved D36 0.40 mm to (255.6, 198.3)
- moved D36 0.25 mm to (179.4, 113.2)
- moved D36 0.25 mm to (160.4, 113.2)
- moved D36 0.25 mm to (198.5, 113.2)
- moved D36 0.23 mm to (217.7, 113.2)
- moved D36 0.12 mm to (279.4, 160.6)
Routing:
- net Col13: track 211.1 -> 183.1 mm
- net Col15: track 173.5 -> 170.7 mm
- net Col19: track 109.3 -> 111.5 mm
- net Row1: track 401.9 -> 403.7 mm
- net Col12: track 178.7 -> 180.3 mm
- net D+: track 80.7 -> 79.2 mm
- net Col5: track 245.4 -> 246.5 mm
- net D-: track 80.7 -> 81.9 mm
- net Col4: track 265.5 -> 266.5 mm
- net Col3: track 309.6 -> 310.5 mm
- net Col2: track 325.6 -> 326.5 mm
- net Col1: track 351.7 -> 352.6 mm
- net Col17: track 175.2 -> 174.7 mm
- net Dbus-: track 59.1 -> 59.7 mm
Other:
- outline, holes or cut-outs redrawn

Commit message: more routing
Parts:
- removed ?: , 
- REF**: value LQFP100-14X14mm -> LQFP100
Connections:
- REF** pad 51: (no net) -> Col10
- REF** pad 52: (no net) -> Row3
- REF** pad 53: (no net) -> Row4
- REF** pad 54: (no net) -> Row5
- REF** pad 63: (no net) -> Row6
- REF** pad 64: (no net) -> Col6
Routing:
- net Row6: track 400.0 -> 486.9 mm, vias 0 -> 2
- net Col6: track 182.0 -> 262.2 mm, vias 0 -> 1
- net Row5: track 409.1 -> 472.6 mm, vias 0 -> 2
- net Row4: track 416.4 -> 457.9 mm, vias 0 -> 2
- net Row3: track 437.7 -> 445.5 mm
- net Col10: track 248.3 -> 253.1 mm, vias 0 -> 1
- net Col9: track 251.5 -> 247.7 mm
- net D+: track 79.2 -> 81.7 mm
