File: EDA/berlin.kicad_pcb (KiCad board)
At the start: 2 copper layers, 431.8 x 173.4 mm, 380 parts, among them J1 TYPE-C-31-M12_13, SW1,1 Rotary_Encoder_Switch_Chassis, SW1,10 MXSwitch, SW1,11 MXSwitch, SW1,12 MXSwitch, SW1,13 MXSwitch, SW1,14 MXSwitch, SW1,15 MXSwitch, SW1,16 Rotary_Encoder_Switch_Chassis, SW1,2 MXSwitch, SW1,3 MXSwitch, SW1,4 MXSwitch, SW1,5 MXSwitch, SW1,6 MXSwitch, SW1,7 MXSwitch, SW1,8 MXSwitch, SW1,9 MXSwitch, SW2,1 MXSwitch, SW2,10 MXSwitch, SW2,11 MXSwitch, SW2,12 MXSwitch, SW2,13 MXSwitch, SW2,14 MXSwitch, SW2,15 MXSwitch, SW2,16 MXSwitch, SW2,17 MXSwitch, SW2,18 MXSwitch, SW2,19 2,19, SW2,2 MXSwitch, SW2,3 MXSwitch, SW2,4 MXSwitch, SW2,5 MXSwitch, SW2,6 MXSwitch, SW2,7 MXSwitch, SW2,8 MXSwitch, SW2,9 MXSwitch, SW3,1 MXSwitch, SW3,10 MXSwitch, SW3,11 MXSwitch, SW3,12 MXSwitch, SW3,13 MXSwitch, SW3,14 MXSwitch, SW3,15 MXSwitch, SW3,16 MXSwitch, SW3,17 MXSwitch, SW3,18 MXSwitch, SW3,19 MXSwitch, SW3,2 MXSwitch, SW3,3 MXSwitch, SW3,4 MXSwitch, SW3,5 MXSwitch, SW3,6 MXSwitch, SW3,7 MXSwitch, SW3,8 MXSwitch, SW3,9 MXSwitch, SW4,1 MXSwitch, SW4,10 MXSwitch, SW4,11 MXSwitch, SW4,12 MXSwitch, SW4,13 MXSwitch, SW4,14 MXSwitch, SW4,15 MXSwitch, SW4,16 MXSwitch, SW4,17 MXSwitch, SW4,18 MXSwitch, SW4,19 MXSwitch, SW4,2 MXSwitch, SW4,3 MXSwitch, SW4,4 MXSwitch, SW4,5 MXSwitch, SW4,6 MXSwitch, SW4,7 MXSwitch, SW4,8 MXSwitch, SW4,9 MXSwitch, SW5,1 MXSwitch, SW5,10 MXSwitch, SW5,11 MXSwitch, SW5,12 MXSwitch, SW5,13 MXSwitch, SW5,14 MXSwitch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

Commit message: route jtag and last key traces
Parts:
- added J2: Conn_01x14, acheron_Connectors:Conn_ARM_JTAG_SWD_10, F.Cu at (234.0, 69.5)
- D94 (x3): moved to F.Cu
- moved D94 3.48 mm to (240.7, 133.0)
- moved D94 3.00 mm to (259.8, 132.4)
- moved D94 2.17 mm to (421.7, 131.0)
- moved D94 2.09 mm to (383.7, 131.1)
- moved D94 1.65 mm to (403.3, 131.0)
- moved D94 1.24 mm to (36.8, 70.5)
Connections:
- REF** pad 14: (no net) -> NRST
- REF** pad 15: (no net) -> Col16
- REF** pad 16: (no net) -> Col19
- REF** pad 17: (no net) -> Col18
- REF** pad 18: (no net) -> Col17
- REF** pad 20: (no net) -> GND
- REF** pad 27: (no net) -> GND
- REF** pad 33: (no net) -> Col15
- REF** pad 34: (no net) -> Col14
- REF** pad 35: (no net) -> Col13
- REF** pad 37: (no net) -> Col12
- REF** pad 47: (no net) -> Col11
- REF** pad 48: (no net) -> Row7
- REF** pad 49: (no net) -> GND
- REF** pad 72: (no net) -> SWDIO
- REF** pad 74: (no net) -> GND
- REF** pad 76: (no net) -> SWCLK
- REF** pad 94: (no net) -> BOOT0
- REF** pad 99: (no net) -> GND
Routing:
- net Col19: track 111.5 -> 309.0 mm
- net Col18: track 155.5 -> 333.7 mm
- net Col17: track 174.7 -> 333.6 mm
- net Col16: track 161.3 -> 298.1 mm
- net Col15: track 170.7 -> 292.2 mm, vias 0 -> 1
- net Col14: track 167.3 -> 270.3 mm, vias 0 -> 1
- net Row7: track 414.4 -> 499.7 mm, vias 0 -> 2
- net SWDIO: track 0.00 -> 55.9 mm, vias 0 -> 1
- net NRST: track 0.00 -> 49.2 mm, vias 0 -> 1
- net SWCLK: track 0.00 -> 47.8 mm, vias 0 -> 1
- net Col13: track 183.1 -> 223.0 mm, vias 0 -> 1
- net Col12: track 180.3 -> 202.8 mm, vias 0 -> 1
- net (no net): track 871.0 -> 890.1 mm, vias 0 -> 1
- net Col11: track 245.7 -> 254.1 mm, vias 0 -> 1
- net Col10: track 253.1 -> 258.7 mm, vias 1 -> 2
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
Commit message: update drc
Routing:
- net (no net): track 890.1 -> 885.8 mm
- net Row3: track 446.6 -> 445.3 mm
Changed lines of the file:
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@@
     (property "Sheetname" "")
     (attr smd)
-    (fp_text reference "D94" (at -0.00012 -1.7786 -90) (layer "B.SilkS")
+    (fp_text reference "D94" (at -0.762 -2.0828) (layer "B.SilkS")
       (effects (font (size 0.6 0.6) (thickness 0.15)) (justify mirror))
     )
@@
     (property "Sheetname" "")
     (attr smd)
-    (fp_text reference "D94" (at -0.00012 -1.7786 -90) (layer "B.SilkS")
+    (fp_text reference "D94" (at -0.2032 -2.0574) (layer "B.SilkS")
       (effects (font (size 0.6 0.6) (thickness 0.15)) (justify mirror))
     )
@@
     (property "Sheetname" "")
     (attr smd)
-    (fp_text reference "D94" (at -0.00012 -1.7786) (layer "B.SilkS")
+    (fp_text reference "D94" (at -0.00012 1.7526) (layer "B.SilkS")
       (effects (font (size 0.6 0.6) (thickness 0.15)) (justify mirror))
     )
@@
   (segment (start 142.20825 153.06675) (end 138.65225 153.06675) (width 0.2) (layer "B.Cu") (net 0))
   (segment (start 213.64575 191.16675) (end 210.08975 191.16675) (width 0.2) (layer "B.Cu") (net 0))
-  (segment (start 385.572 133.31825) (end 386.30225 134.0485) (width 0.25) (layer "B.Cu") (net 0))
   (segment (start 424.40225 134.0485) (end 427.95825 134.0485) (width 0.2) (layer "B.Cu") (net 0))
   (segment (start 59.182 208.152) (end 59.182 209.32775) (width 0.25) (layer "B.Cu") (net 0))
@@
   (segment (start 119.60225 86.39175) (end 123.15825 86.39175) (width 0.2) (layer "B.Cu") (net 0))
   (segment (start 423.672 171.41825) (end 424.40225 172.1485) (width 0.25) (layer "B.Cu") (net 0))
-  (segment (start 404.622 133.31825) (end 405.35225 134.0485) (width 0.25) (layer "B.Cu") (net 0))
   (segment (start 81.50225 151.09825) (end 81.152 150.748) (width 0.2) (layer "B.Cu") (net 0))
   (segment (start 299.72 85.5345) (end 300.57725 86.39175) (width 0.25) (layer "B.Cu") (net 0))
@@
   (segment (start 242.57 83.565) (end 242.57 85.53434) (width 0.25) (layer "B.Cu") (net 0))
   (segment (start 33.87725 134.01675) (end 37.43325 134.01675) (width 0.25) (layer "B.Cu") (net 0))
-  (segment (start 242.57 133.1595) (end 243.42725 134.01675) (width 0.25) (layer "B.Cu") (net 0))
   (segment (start 386.30225 172.1485) (end 389.85825 172.1485) (width 0.25) (layer "B.Cu") (net 0))
   (segment (start 52.92725 134.01675) (end 56.48325 134.01675) (width 0.25) (layer "B.Cu") (net 0))
@@
   (segment (start 291.05225 130.60275) (end 294.025 127.63) (width 0.2) (layer "B.Cu") (net 0))
   (segment (start 172.085 105.44175) (end 175.641 105.44175) (width 0.25) (layer "B.Cu") (net 0))
-  (segment (start 423.672 133.31825) (end 424.40225 134.0485) (width 0.25) (layer "B.Cu") (net 0))
   (segment (start 33.02 133.1595) (end 33.87725 134.01675) (width 0.25) (layer "B.Cu") (net 0))
   (segment (start 243.42741 86.39175) (end 246.98341 86.39175) (width 0.25) (layer "B.Cu") (net 0))
@@
   (segment (start 403.3012 129.3886) (end 403.296589 129.383989) (width 0.25) (layer "F.Cu") (net 11))
   (segment (start 383.7432 104.9782) (end 383.7432 129.414) (width 0.25) (layer "F.Cu") (net 11))
-  (segment (start 379.857 101.092) (end 378.968 100.203) (width 0.25) (layer "F.Cu") (net 11))
   (segment (start 403.296589 129.383989) (end 383.773211 129.383989) (width 0.25) (layer "F.Cu") (net 11))
   (via (at 379.857 101.092) (size 0.8) (drill 0.4) (layers "F.Cu" "B.Cu") (net 11))

Commit message: small updates in naming/routing
Parts:
- added L702: L_Core_Ferrite, Inductor_SMD:L_0805_2012Metric_Pad1.15x1.40mm_HandSolder, B.Cu at (150.0, 58.2)
- added R705: 5.1k, Resistor_SMD:R_0805_2012Metric_Pad1.15x1.40mm_HandSolder, B.Cu at (146.9, 61.8)
- added R706: 5.1k, Resistor_SMD:R_0805_2012Metric_Pad1.15x1.40mm_HandSolder, B.Cu at (139.2, 62.4)
- moved U702 32.7 mm to (138.4, 93.4), turned to -90 degrees
- renumbered D94 to D1, D94 to D2, D94 to D3, D94 to D4, D94 to D5, D94 to D6, D94 to D7
Connections:
- J1 pad A1: (no net) -> GND
- J1 pad A4: (no net) -> VBUS
- J1 pad A5: (no net) -> CC1
- J1 pad A8: (no net) -> SBU1
- J1 pad B1: (no net) -> GND
- J1 pad B4: (no net) -> VBUS
- J1 pad B5: (no net) -> CC2
- J1 pad B8: (no net) -> SBU2
- J1 pad S: (no net) -> S
- REF** pad 1: (no net) -> GND
- REF** pad 3: (no net) -> Pcomp1
- REF** pad MP: (no net) -> GND
- U702 pad 1: (no net) -> 3V3
- U702 pad 2: (no net) -> 5V
- U702 pad 3: (no net) -> 5V
- U702 pad 4: (no net) -> GND
Routing:
- net VBUS: track 0.00 -> 59.3 mm, vias 0 -> 4
- net CC1: track 0.00 -> 6.42 mm
- net CC2: track 0.00 -> 5.19 mm
- net Dbus-: track 59.7 -> 58.1 mm
- added copper zone on B.Cu, net S
- added copper zone on B.Cu, net VBUS
- added copper zone on F.Cu, net VBUS
Other:
- outline, holes or cut-outs redrawn
