File: EDA/berlin.kicad_sch (KiCad schematic)
At the start: 615 parts, among them J1 TYPE-C-31-M12_13, J2 Conn_ARM_JTAG_SWD_10, Q701 DTC123J, SW1,1 Rotary_Encoder_Switch_Chassis, SW1,10 MXSwitch, SW1,11 MXSwitch, SW1,12 MXSwitch, SW1,13 MXSwitch, SW1,14 MXSwitch, SW1,15 MXSwitch, SW1,16 Rotary_Encoder_Switch_Chassis, SW1,2 MXSwitch, SW1,3 MXSwitch, SW1,4 MXSwitch, SW1,5 MXSwitch, SW1,6 MXSwitch, SW1,7 MXSwitch, SW1,8 MXSwitch, SW1,9 MXSwitch, SW2,1 MXSwitch, SW2,10 MXSwitch, SW2,11 MXSwitch, SW2,12 MXSwitch, SW2,13 MXSwitch, SW2,14 MXSwitch, SW2,15 MXSwitch, SW2,16 MXSwitch, SW2,17 MXSwitch, SW2,18 MXSwitch, SW2,19 MXSwitch, SW2,2 MXSwitch, SW2,3 MXSwitch, SW2,4 MXSwitch, SW2,5 MXSwitch, SW2,6 MXSwitch, SW2,7 MXSwitch, SW2,9 MXSwitch, SW20-7,3 MXSwitch, SW200 SW_Push, SW3,1 MXSwitch, SW3,10 MXSwitch, SW3,11 MXSwitch, SW3,12 MXSwitch, SW3,13 MXSwitch, SW3,14 MXSwitch, SW3,15 MXSwitch, SW3,16 MXSwitch, SW3,17 MXSwitch, SW3,18 MXSwitch, SW3,19 MXSwitch, SW3,2 MXSwitch, SW3,3 MXSwitch, SW3,4 MXSwitch, SW3,5 MXSwitch, SW3,6 MXSwitch, SW3,7 MXSwitch, SW3,8 MXSwitch, SW3,9 MXSwitch, SW39-7,6 MXSwitch, SW4,1 MXSwitch, SW4,10 MXSwitch, SW4,11 MXSwitch, SW4,12 MXSwitch, SW4,13 MXSwitch, SW4,14 MXSwitch, SW4,15 MXSwitch, SW4,16 MXSwitch, SW4,17 MXSwitch, SW4,18 MXSwitch, SW4,19 MXSwitch, SW4,2 MXSwitch, SW4,3 MXSwitch, SW4,4 MXSwitch, SW4,5 MXSwitch, SW4,6 MXSwitch, SW4,7 MXSwitch, SW4,8 MXSwitch, SW4,9 MXSwitch, SW5,1 MXSwitch, SW5,10 MXSwitch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

Commit message: annotated diodes next to switches
Parts:
- removed R? (x3): 330, Resistor_THT:R_Axial_DIN0207_L6.3mm_D2.5mm_P7.62mm_Horizontal, symbol Device:R
- removed R? (x2): 10k, Resistor_SMD:R_0805_2012Metric_Pad1.15x1.40mm_HandSolder, symbol Device:R
- removed U?: STM32F072CBTx, Package_QFP:LQFP-48_7x7mm_P0.5mm, symbol MCU_ST_STM32F0:STM32F072CBTx
- removed UA?: STM32F072CBUx, Package_DFN_QFN:QFN-48-1EP_7x7mm_P0.5mm_EP5.6x5.6mm, symbol MCU_ST_STM32F0:STM32F072CBUx
- gave numbers to parts that had none: 119
- renumbered SW6-7,1 to SW7,1, SW20-7,3 to SW7,3, SW39-7,6 to SW7,6, SW64-7,8 to SW7,8, SW64-7,9 to SW7,9
Connections:
- net Row3: now also D97.1 (K)
Other:
- note removed: "LQFP-48"
- note removed: "UFQFPN48 alternate"

Commit message: fix rotary encoders
Connections:
- net Col1: now also SW1,1.3 (SW); no longer SW1,1.S1
- net Col16: now also SW1,16.3 (SW); no longer SW1,16.S1
- net EncA: no longer SW1,1.A, SW1,16.A
- net EncB: no longer SW1,1.B, SW1,16.B
- net at D1.2 (A): now also SW1,1.5 (Common_+); no longer SW1,1.S2
- net at D102.2 (A): now also SW1,16.5 (Common_+); no longer SW1,16.S2
- new net 1,1 B: SW1,1.4 (B)
- new net 1,1 G: SW1,1.2 (G)
- new net 1,1 R: SW1,1.1 (R)
- new net 1,16 B: SW1,16.4 (B)
- new net 1,16 G: SW1,16.2 (G)
- new net 1,16 R: SW1,16.1 (R)
- new net Enc1A: SW1,1.A
- new net Enc1B: SW1,1.B
- new net Enc2A: SW1,16.A
- new net Enc2B: SW1,16.B
Other:
- moved on the sheet: D102, L2

Commit message: update to FT io and LED update
Parts:
- added LED1,1, LED1,16: WS2811S, MSOP8_WDS, symbol 2022-03-27_15-42-26:WS2811S
- added LED1,10, LED1,11, LED1,12, LED1,13, LED1,14, LED1,15, LED1,2, LED1,3, LED1,4, LED1,5, LED1,6, LED1,7, LED1,8, LED1,9: SK6812MINI-E, acheron_Components:SK6812MINI_3535_6028_3.2x2.8mm_Round, symbol 2022-03-27_15-42-261:SK6812MINI-E
Connections:
- net +5V: now also LED1,1.8 (VDD), LED1,10.1 (VDD), LED1,11.1 (VDD), LED1,12.1 (VDD), LED1,13.1 (VDD), LED1,14.1 (VDD), LED1,15.1 (VDD), LED1,16.8 (VDD), LED1,2.1 (VDD), LED1,3.1 (VDD), LED1,4.1 (VDD), LED1,5.1 (VDD), LED1,6.1 (VDD), LED1,7.1 (VDD), LED1,8.1 (VDD), LED1,9.1 (VDD)
- net 1,1 B: now also LED1,1.3 (OUTB)
- net 1,1 G: now also LED1,1.2 (OUTG)
- net 1,1 R: now also LED1,1.1 (OUTR)
- net 1,16 B: now also LED1,16.3 (OUTB)
- net 1,16 G: now also LED1,16.2 (OUTG)
- net 1,16 R: now also LED1,16.1 (OUTR)
- net Col16: now also U1001.11 (PF10); no longer U1001.15 (PC0)
- net GND: now also LED1,1.4 (GND), LED1,10.3 (VSS), LED1,11.3 (VSS), LED1,12.3 (VSS), LED1,13.3 (VSS), LED1,14.3 (VSS), LED1,15.3 (VSS), LED1,16.4 (GND), LED1,2.3 (VSS), LED1,3.3 (VSS), LED1,4.3 (VSS), LED1,5.3 (VSS), LED1,6.3 (VSS), LED1,7.3 (VSS), LED1,8.3 (VSS), LED1,9.3 (VSS)
- new net: LED1,13.2 (DOUT), LED1,14.4 (DIN)
- new net: LED1,12.2 (DOUT), LED1,13.4 (DIN)
- new net: LED1,6.2 (DOUT), LED1,7.4 (DIN)
- new net: LED1,5.2 (DOUT), LED1,6.4 (DIN)
- new net: LED1,3.2 (DOUT), LED1,4.4 (DIN)
- new net: LED1,2.2 (DOUT), LED1,3.4 (DIN)
- new net: LED1,15.2 (DOUT), LED1,16.6 (DIN)
- new net: LED1,1.5 (DO), LED1,2.4 (DIN)
- new net: LED1,8.2 (DOUT), LED1,9.4 (DIN)
- new net: LED1,7.2 (DOUT), LED1,8.4 (DIN)
- new net: LED1,4.2 (DOUT), LED1,5.4 (DIN)
- new net: LED1,11.2 (DOUT), LED1,12.4 (DIN)
- new net: LED1,10.2 (DOUT), LED1,11.4 (DIN)
- new net: LED1,10.4 (DIN), LED1,9.2 (DOUT)
- new net: LED1,14.2 (DOUT), LED1,15.4 (DIN)
- new net LED1: LED1,1.6 (DIN)
- no-connect marks 4 -> 5

Commit message: fix glitchy matrix design
Parts:
- removed D1, D102: 1N4148, acheronComponents:D_SOD-123, symbol Diode:1N4148
Connections:
- net +5V: now also SW1,1.5 (Common_+), SW1,16.5 (Common_+)
- net Col1: no longer SW1,1.3 (SW)
- net Col16: no longer SW1,16.3 (SW)
- new net 1,1 INTERRUPT: SW1,1.3 (SW), SW1,16.3 (SW)
Other:
- moved on the sheet: L1, L2, SW1,1, SW1,16

Commit message: minor led additions
Parts:
- added LED2,1, LED2,10, LED2,11, LED2,12, LED2,13, LED2,14, LED2,15, LED2,16, LED2,17, LED2,18, LED2,19, LED2,2, LED2,3, LED2,4, LED2,5, LED2,6, LED2,7, LED2,8, LED2,9, LED3,1, LED3,10, LED3,11, LED3,12, LED3,13, LED3,14, LED3,15, LED3,16, LED3,17, LED3,18, LED3,19, LED3,2, LED3,3, LED3,4, LED3,5, LED3,6, LED3,7, LED3,8, LED3,9, LED4,1, LED4,10, LED4,11, LED4,12, LED4,13, LED4,14, LED4,15, LED4,16, LED4,17, LED4,18, LED4,19, LED4,2, LED4,3, LED4,4, LED4,5, LED4,6, LED4,7, LED4,8, LED4,9: SK6812MINI-E, acheron_Components:SK6812MINI_3535_6028_3.2x2.8mm_Round, symbol 2022-03-27_15-42-261:SK6812MINI-E
- LED1,10, LED1,11, LED1,12, LED1,13, LED1,14, LED1,15, LED1,2, LED1,3, LED1,4, LED1,5, LED1,6, LED1,7, LED1,8, LED1,9: MFN Dongguan Opsco Optoelectronics -> (none)
Connections:
- net +5V: now also LED2,1.1 (VDD), LED2,10.1 (VDD), LED2,11.1 (VDD), LED2,12.1 (VDD), LED2,13.1 (VDD), LED2,14.1 (VDD), LED2,15.1 (VDD), LED2,16.1 (VDD), LED2,17.1 (VDD), LED2,18.1 (VDD), LED2,19.1 (VDD), LED2,2.1 (VDD), LED2,3.1 (VDD), LED2,4.1 (VDD), LED2,5.1 (VDD), LED2,6.1 (VDD), LED2,7.1 (VDD), LED2,8.1 (VDD), LED2,9.1 (VDD), LED3,1.1 (VDD), LED3,10.1 (VDD), LED3,11.1 (VDD), LED3,12.1 (VDD), LED3,13.1 (VDD), LED3,14.1 (VDD), LED3,15.1 (VDD), LED3,16.1 (VDD), LED3,17.1 (VDD), LED3,18.1 (VDD), LED3,19.1 (VDD), LED3,2.1 (VDD), LED3,3.1 (VDD), LED3,4.1 (VDD), LED3,5.1 (VDD), LED3,6.1 (VDD), LED3,7.1 (VDD), LED3,8.1 (VDD), LED3,9.1 (VDD), LED4,1.1 (VDD), LED4,10.1 (VDD), LED4,11.1 (VDD), LED4,12.1 (VDD), LED4,13.1 (VDD), LED4,14.1 (VDD), LED4,15.1 (VDD), LED4,16.1 (VDD), LED4,17.1 (VDD), LED4,18.1 (VDD), LED4,19.1 (VDD), LED4,2.1 (VDD), LED4,3.1 (VDD), LED4,4.1 (VDD), LED4,5.1 (VDD), LED4,6.1 (VDD), LED4,7.1 (VDD), LED4,8.1 (VDD), LED4,9.1 (VDD)
- net GND: now also LED2,1.3 (VSS), LED2,10.3 (VSS), LED2,11.3 (VSS), LED2,12.3 (VSS), LED2,13.3 (VSS), LED2,14.3 (VSS), LED2,15.3 (VSS), LED2,16.3 (VSS), LED2,17.3 (VSS), LED2,18.3 (VSS), LED2,19.3 (VSS), LED2,2.3 (VSS), LED2,3.3 (VSS), LED2,4.3 (VSS), LED2,5.3 (VSS), LED2,6.3 (VSS), LED2,7.3 (VSS), LED2,8.3 (VSS), LED2,9.3 (VSS), LED3,1.3 (VSS), LED3,10.3 (VSS), LED3,11.3 (VSS), LED3,12.3 (VSS), LED3,13.3 (VSS), LED3,14.3 (VSS), LED3,15.3 (VSS), LED3,16.3 (VSS), LED3,17.3 (VSS), LED3,18.3 (VSS), LED3,19.3 (VSS), LED3,2.3 (VSS), LED3,3.3 (VSS), LED3,4.3 (VSS), LED3,5.3 (VSS), LED3,6.3 (VSS), LED3,7.3 (VSS), LED3,8.3 (VSS), LED3,9.3 (VSS), LED4,1.3 (VSS), LED4,10.3 (VSS), LED4,11.3 (VSS), LED4,12.3 (VSS), LED4,13.3 (VSS), LED4,14.3 (VSS), LED4,15.3 (VSS), LED4,16.3 (VSS), LED4,17.3 (VSS), LED4,18.3 (VSS), LED4,19.3 (VSS), LED4,2.3 (VSS), LED4,3.3 (VSS), LED4,4.3 (VSS), LED4,5.3 (VSS), LED4,6.3 (VSS), LED4,7.3 (VSS), LED4,8.3 (VSS), LED4,9.3 (VSS)
- new net: LED4,6.2 (DOUT), LED4,7.4 (DIN)
- new net: LED4,5.2 (DOUT), LED4,6.4 (DIN)
- new net: LED4,15.2 (DOUT), LED4,16.4 (DIN)
- new net: LED4,14.2 (DOUT), LED4,15.4 (DIN)
- new net: LED2,7.2 (DOUT), LED2,8.4 (DIN)
- new net: LED2,6.2 (DOUT), LED2,7.4 (DIN)
- new net: LED4,16.2 (DOUT), LED4,17.4 (DIN)
- new net: LED2,2.2 (DOUT), LED2,3.4 (DIN)
- new net: LED2,1.2 (DOUT), LED2,2.4 (DIN)
- new net: LED3,8.2 (DOUT), LED3,9.4 (DIN)
- new net: LED3,7.2 (DOUT), LED3,8.4 (DIN)
- new net: LED4,17.2 (DOUT), LED4,18.4 (DIN)
- new net: LED2,8.2 (DOUT), LED2,9.4 (DIN)
- new net: LED4,1.2 (DOUT), LED4,2.4 (DIN)
- new net: LED3,5.2 (DOUT), LED3,6.4 (DIN)
- new net: LED3,4.2 (DOUT), LED3,5.4 (DIN)
- new net: LED2,12.2 (DOUT), LED2,13.4 (DIN)
- new net: LED2,11.2 (DOUT), LED2,12.4 (DIN)
- new net: LED3,11.2 (DOUT), LED3,12.4 (DIN)
- new net: LED3,10.2 (DOUT), LED3,11.4 (DIN)
- new net: LED2,10.2 (DOUT), LED2,11.4 (DIN)
- new net: LED4,2.2 (DOUT), LED4,3.4 (DIN)
- new net: LED3,14.2 (DOUT), LED3,15.4 (DIN)
- new net: LED3,13.2 (DOUT), LED3,14.4 (DIN)
- new net: LED3,3.2 (DOUT), LED3,4.4 (DIN)
- new net: LED3,2.2 (DOUT), LED3,3.4 (DIN)
- new net: LED3,12.2 (DOUT), LED3,13.4 (DIN)
- new net: LED4,10.2 (DOUT), LED4,11.4 (DIN)
- new net: LED4,10.4 (DIN), LED4,9.2 (DOUT)
- new net: LED4,13.2 (DOUT), LED4,14.4 (DIN)
- new net: LED4,12.2 (DOUT), LED4,13.4 (DIN)
- new net: LED3,16.2 (DOUT), LED3,17.4 (DIN)
- new net: LED3,15.2 (DOUT), LED3,16.4 (DIN)
- new net: LED4,4.2 (DOUT), LED4,5.4 (DIN)
- new net: LED4,3.2 (DOUT), LED4,4.4 (DIN)
- new net: LED2,14.2 (DOUT), LED2,15.4 (DIN)
- new net: LED2,13.2 (DOUT), LED2,14.4 (DIN)
- new net: LED3,10.4 (DIN), LED3,9.2 (DOUT)
- new net: LED3,18.2 (DOUT), LED3,19.4 (DIN)
- new net: LED3,17.2 (DOUT), LED3,18.4 (DIN)
- new net: LED2,4.2 (DOUT), LED2,5.4 (DIN)
- new net: LED2,3.2 (DOUT), LED2,4.4 (DIN)
- new net: LED2,17.2 (DOUT), LED2,18.4 (DIN)
- new net: LED2,16.2 (DOUT), LED2,17.4 (DIN)
- new net: LED2,15.2 (DOUT), LED2,16.4 (DIN)
- new net: LED3,1.2 (DOUT), LED3,2.4 (DIN)
- new net: LED3,6.2 (DOUT), LED3,7.4 (DIN)
- new net: LED4,8.2 (DOUT), LED4,9.4 (DIN)
- new net: LED2,5.2 (DOUT), LED2,6.4 (DIN)
- new net: LED2,10.4 (DIN), LED2,9.2 (DOUT)
- new net: LED4,18.2 (DOUT), LED4,19.4 (DIN)
- new net: LED2,18.2 (DOUT), LED2,19.4 (DIN)
- new net: LED4,7.2 (DOUT), LED4,8.4 (DIN)
- new net: LED4,11.2 (DOUT), LED4,12.4 (DIN)

Commit message: reformatting/reannotation, add new display mockup
Parts:
- added C101, C102: 100n, Capacitor_SMD:C_1206_3216Metric_Pad1.42x1.75mm_HandSolder, symbol Device:C
- added R101, R102: 33, Resistor_SMD:R_0805_2012Metric_Pad1.15x1.40mm_HandSolder, symbol Device:R
- renumbered J1 to J201, J2 to J202, SW200 to SW201, U1001 to U501, U3 to U701
Connections:
- net +5V: now also R101.1, R102.1; no longer LED1,1.8 (VDD), LED1,16.8 (VDD)
- net GND: now also C101.2, C102.2
- new net: C102.1, LED1,16.8 (VDD), R102.2
- new net: C101.1, LED1,1.8 (VDD), R101.2
Other:
- note added: "Component annotation keys: Type Shortcut+Usage Number+Part number(max. 100 parts) Usage Number: 1-Auxiliary components for matrix 2-interface components 3-auxiliary components for logic (e.g. pullups) 5-logic/ic components 7-power delivery components notes: components inside the matrix layout are assigned [type]+[row],[column] diodes in the matrix are labelled iteratively because of sheer numbers"
- moved on the sheet: C701, C703, C704, C705, C706, C707, C708, C709, C710, C711, C715, C717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

Commit message: add&annotate all leds
Parts:
- added LED5,1, LED5,10, LED5,11, LED5,12, LED5,13, LED5,14, LED5,15, LED5,16, LED5,17, LED5,18, LED5,19, LED5,2, LED5,3, LED5,4, LED5,5, LED5,6, LED5,7, LED5,8, LED5,9, LED6,1, LED6,10, LED6,11, LED6,12, LED6,13, LED6,15, LED6,17, LED6,18, LED6,19, LED6,2, LED6,3, LED6,4, LED6,5, LED6,6, LED6,7, LED6,8, LED6,9, LED7,1, LED7,10, LED7,11, LED7,12, LED7,13, LED7,14, LED7,15, LED7,16, LED7,17, LED7,18, LED7,2, LED7,3, LED7,5, LED7,6, LED7,7, LED7,8, LED7,9: SK6812MINI-E, acheron_Components:SK6812MINI_3535_6028_3.2x2.8mm_Round, symbol 2022-03-27_15-42-261:SK6812MINI-E
Connections:
- net +5V: now also LED5,1.1 (VDD), LED5,10.1 (VDD), LED5,11.1 (VDD), LED5,12.1 (VDD), LED5,13.1 (VDD), LED5,14.1 (VDD), LED5,15.1 (VDD), LED5,16.1 (VDD), LED5,17.1 (VDD), LED5,18.1 (VDD), LED5,19.1 (VDD), LED5,2.1 (VDD), LED5,3.1 (VDD), LED5,4.1 (VDD), LED5,5.1 (VDD), LED5,6.1 (VDD), LED5,7.1 (VDD), LED5,8.1 (VDD), LED5,9.1 (VDD), LED6,1.1 (VDD), LED6,10.1 (VDD), LED6,11.1 (VDD), LED6,12.1 (VDD), LED6,13.1 (VDD), LED6,15.1 (VDD), LED6,17.1 (VDD), LED6,18.1 (VDD), LED6,19.1 (VDD), LED6,2.1 (VDD), LED6,3.1 (VDD), LED6,4.1 (VDD), LED6,5.1 (VDD), LED6,6.1 (VDD), LED6,7.1 (VDD), LED6,8.1 (VDD), LED6,9.1 (VDD), LED7,1.1 (VDD), LED7,10.1 (VDD), LED7,11.1 (VDD), LED7,12.1 (VDD), LED7,13.1 (VDD), LED7,14.1 (VDD), LED7,15.1 (VDD), LED7,16.1 (VDD), LED7,17.1 (VDD), LED7,18.1 (VDD), LED7,2.1 (VDD), LED7,3.1 (VDD), LED7,5.1 (VDD), LED7,6.1 (VDD), LED7,7.1 (VDD), LED7,8.1 (VDD), LED7,9.1 (VDD)
- net GND: now also LED5,1.3 (VSS), LED5,10.3 (VSS), LED5,11.3 (VSS), LED5,12.3 (VSS), LED5,13.3 (VSS), LED5,14.3 (VSS), LED5,15.3 (VSS), LED5,16.3 (VSS), LED5,17.3 (VSS), LED5,18.3 (VSS), LED5,19.3 (VSS), LED5,2.3 (VSS), LED5,3.3 (VSS), LED5,4.3 (VSS), LED5,5.3 (VSS), LED5,6.3 (VSS), LED5,7.3 (VSS), LED5,8.3 (VSS), LED5,9.3 (VSS), LED6,1.3 (VSS), LED6,10.3 (VSS), LED6,11.3 (VSS), LED6,12.3 (VSS), LED6,13.3 (VSS), LED6,15.3 (VSS), LED6,17.3 (VSS), LED6,18.3 (VSS), LED6,19.3 (VSS), LED6,2.3 (VSS), LED6,3.3 (VSS), LED6,4.3 (VSS), LED6,5.3 (VSS), LED6,6.3 (VSS), LED6,7.3 (VSS), LED6,8.3 (VSS), LED6,9.3 (VSS), LED7,1.3 (VSS), LED7,10.3 (VSS), LED7,11.3 (VSS), LED7,12.3 (VSS), LED7,13.3 (VSS), LED7,14.3 (VSS), LED7,15.3 (VSS), LED7,16.3 (VSS), LED7,17.3 (VSS), LED7,18.3 (VSS), LED7,2.3 (VSS), LED7,3.3 (VSS), LED7,5.3 (VSS), LED7,6.3 (VSS), LED7,7.3 (VSS), LED7,8.3 (VSS), LED7,9.3 (VSS)
- net LED4: now reaches LED4,1.4 (DIN)
- net LED3: now reaches LED3,1.4 (DIN)
- net LED2: now reaches LED2,1.4 (DIN)
- new net: LED5,8.2 (DOUT), LED5,9.4 (DIN)
- new net: LED5,7.2 (DOUT), LED5,8.4 (DIN)
- new net: LED7,17.2 (DOUT), LED7,18.4 (DIN)
- new net: LED7,16.2 (DOUT), LED7,17.4 (DIN)
- new net: LED7,15.2 (DOUT), LED7,16.4 (DIN)
- new net: LED5,6.2 (DOUT), LED5,7.4 (DIN)
- new net: LED5,5.2 (DOUT), LED5,6.4 (DIN)
- new net: LED7,11.2 (DOUT), LED7,12.4 (DIN)
- new net: LED7,10.2 (DOUT), LED7,11.4 (DIN)
- new net: LED6,12.2 (DOUT), LED6,13.4 (DIN)
- new net: LED6,11.2 (DOUT), LED6,12.4 (DIN)
- new net: LED6,17.2 (DOUT), LED6,18.4 (DIN)
- new net: LED6,15.2 (DOUT), LED6,17.4 (DIN)
- new net: LED5,3.2 (DOUT), LED5,4.4 (DIN)
- new net: LED5,2.2 (DOUT), LED5,3.4 (DIN)
- new net: LED7,2.2 (DOUT), LED7,3.4 (DIN)
- new net: LED7,1.2 (DOUT), LED7,2.4 (DIN)
- new net: LED5,13.2 (DOUT), LED5,14.4 (DIN)
- new net: LED5,12.2 (DOUT), LED5,13.4 (DIN)
- new net: LED5,10.4 (DIN), LED5,9.2 (DOUT)
- new net: LED5,17.2 (DOUT), LED5,18.4 (DIN)
- new net: LED5,16.2 (DOUT), LED5,17.4 (DIN)
- new net: LED5,1.2 (DOUT), LED5,2.4 (DIN)
- new net: LED5,11.2 (DOUT), LED5,12.4 (DIN)
- new net: LED5,10.2 (DOUT), LED5,11.4 (DIN)
- new net: LED7,12.2 (DOUT), LED7,13.4 (DIN)
- new net: LED7,3.2 (DOUT), LED7,5.4 (DIN)
- new net: LED6,13.2 (DOUT), LED6,15.4 (DIN)
- new net: LED5,18.2 (DOUT), LED5,19.4 (DIN)
- new net: LED6,10.2 (DOUT), LED6,11.4 (DIN)
- new net: LED6,6.2 (DOUT), LED6,7.4 (DIN)
- new net: LED6,5.2 (DOUT), LED6,6.4 (DIN)
- new net: LED6,1.2 (DOUT), LED6,2.4 (DIN)
- new net: LED7,5.2 (DOUT), LED7,6.4 (DIN)
- new net: LED6,7.2 (DOUT), LED6,8.4 (DIN)
- new net: LED7,8.2 (DOUT), LED7,9.4 (DIN)
- new net: LED7,7.2 (DOUT), LED7,8.4 (DIN)
- new net: LED7,10.4 (DIN), LED7,9.2 (DOUT)
- new net: LED5,14.2 (DOUT), LED5,15.4 (DIN)
- new net: LED7,13.2 (DOUT), LED7,14.4 (DIN)
- new net: LED6,10.4 (DIN), LED6,9.2 (DOUT)
- new net: LED6,2.2 (DOUT), LED6,3.4 (DIN)
- new net: LED7,14.2 (DOUT), LED7,15.4 (DIN)
- new net: LED5,15.2 (DOUT), LED5,16.4 (DIN)
- new net: LED5,4.2 (DOUT), LED5,5.4 (DIN)
- new net: LED6,4.2 (DOUT), LED6,5.4 (DIN)
- new net: LED6,3.2 (DOUT), LED6,4.4 (DIN)
- new net: LED6,8.2 (DOUT), LED6,9.4 (DIN)
- new net: LED6,18.2 (DOUT), LED6,19.4 (DIN)
- new net: LED7,6.2 (DOUT), LED7,7.4 (DIN)
- new net LED5: LED5,1.4 (DIN)
- new net LED6: LED6,1.4 (DIN)
- new net LED7: LED7,1.4 (DIN)
Other:
- moved on the sheet: C101, C102, LED1,1, LED1,10, LED1,11, LED1,12, LED1,13, LED1,14, LED1,15, LED1,16, LED1,2, LED1,3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

Commit message: minor led changes
Parts:
- added C? (x12): 100nF, Capacitor_SMD:C_0805_2012Metric_Pad1.15x1.40mm_HandSolder, symbol Device:C
- added C? (x2): 10u, Capacitor_SMD:C_1206_3216Metric_Pad1.42x1.75mm_HandSolder, symbol Device:C
Connections:
- net LED3 is gone; now on an unnamed net: LED3,1.4 (DIN)
- net LED4 is gone; now on net LED2: LED4,1.4 (DIN)
- net LED5 is gone; now on an unnamed net: LED5,1.4 (DIN)
- net LED6 is gone; now on an unnamed net: LED6,1.4 (DIN)
- net LED7 is gone; now on an unnamed net: LED7,1.4 (DIN)
- net +5V: now also C?.1, C?.1, C?.1, C?.1, C?.1, C?.1, C?.1, C?.1, C?.1, C?.1, C?.1, C?.1, C?.1, C?.1
- net GND: now also C?.2, C?.2, C?.2, C?.2, C?.2, C?.2, C?.2, C?.2, C?.2, C?.2, C?.2, C?.2, C?.2, C?.2
- net LED2: no longer LED2,1.4 (DIN)
- net at LED1,16.5 (DO): now also LED2,1.4 (DIN)
- no-connect marks 5 -> 4
